Commit message: Recent changes for full waypoint following sim using only gps and imu and wheel encoder

File: urdf/lotus_robot.urdf (robot description, URDF)
Before this commit: robot two_wheeled_robot, 5 links, 4 joints
Links:
- removed link lidar_link
- added link gps_link
Joints:
- removed joint lidar_joint
- added joint gps_joint: type fixed, parent base_link, child gps_link, origin xyz=0.10 0.0 0.05 rpy=0 0 0
