Commit message: Latest

File: urdf/4wd_properties.urdf.xacro (robot description, xacro)
@@ -8,5 +8,5 @@
   <xacro:property name="wheel_width" value="0.04445" />
   <xacro:property name="front_wheel_pos_x" value="0.120" />
-  <xacro:property name="rear_wheel_pos_x" value="0.120" />
+  <xacro:property name="rear_wheel_pos_x" value="-0.120" />
   <xacro:property name="wheel_pos_y" value="0.1355" />
   <xacro:property name="wheel_pos_z" value="-0.04788" />

File: urdf/robots/4wd.urdf.xacro (robot description, xacro)
@@ -1,4 +1,4 @@
 <?xml version="1.0"?>
-<robot name="linorobot2_4wd" xmlns:xacro="http://ros.org/wiki/xacro">
+<robot name="lotus_4wd" xmlns:xacro="http://ros.org/wiki/xacro">
   <xacro:include filename="$(find two_wheeled_robot)/urdf/4wd_properties.urdf.xacro" />
   <xacro:include filename="$(find two_wheeled_robot)/urdf/mech/base.urdf.xacro" />
@@ -6,7 +6,4 @@
   <xacro:include filename="$(find two_wheeled_robot)/urdf/sensors/imu.urdf.xacro" />
   <xacro:include filename="$(find two_wheeled_robot)/urdf/sensors/gps.urdf.xacro" />
-  <xacro:include filename="$(find two_wheeled_robot)/urdf/sensors/generic_laser.urdf.xacro" />
-  <xacro:include filename="$(find two_wheeled_robot)/urdf/sensors/depth_sensor.urdf.xacro" />
-  <xacro:include filename="$(find two_wheeled_robot)/urdf/controllers/skid_steer.urdf.xacro" />
   <xacro:base
     length="${base_length}"
@@ -21,5 +18,5 @@
     radius="${wheel_radius}"
     width="${wheel_width}"
-    pos_x="${wheel_pos_x}"
+    pos_x="${front_wheel_pos_x}"
     pos_y="${wheel_pos_y}"
     pos_z="${wheel_pos_z}"
@@ -30,5 +27,5 @@
     radius="${wheel_radius}"
     width="${wheel_width}"
-    pos_x="${wheel_pos_x}"
+    pos_x="${front_wheel_pos_x}"
     pos_y="${-wheel_pos_y}"
     pos_z="${wheel_pos_z}"
@@ -39,5 +36,5 @@
     radius="${wheel_radius}"
     width="${wheel_width}"
-    pos_x="${-wheel_pos_x}"
+    pos_x="${rear_wheel_pos_x}"
     pos_y="${wheel_pos_y}"
     pos_z="${wheel_pos_z}"
@@ -48,5 +45,5 @@
     radius="${wheel_radius}"
     width="${wheel_width}"
-    pos_x="${-wheel_pos_x}"
+    pos_x="${rear_wheel_pos_x}"
     pos_y="${-wheel_pos_y}"
     pos_z="${wheel_pos_z}"

File: urdf/sensors/gps.urdf.xacro (robot description, xacro)
@@ -5,5 +5,5 @@
       <parent link="base_link"/>
       <child link="gps_link"/>
-      <origin xyz="0 0 0" rpy="0 0 0"/>
+      <origin xyz="-.23 0 0" rpy="0 0 0"/>
     </joint>
   </xacro:macro>

File: urdf/sensors/imu.urdf.xacro (robot description, xacro)
@@ -5,5 +5,5 @@
       <parent link="base_link"/>
       <child link="imu_link"/>
-      <origin xyz="0 0 0" rpy="0 90 0"/>
+      <origin xyz="-.138 0 .02" rpy="0 1.57 0"/>
     </joint>
   </xacro:macro>
