Commit message: Robot working to some extent

File: urdf/sensors/imu.urdf.xacro (robot description, xacro)
@@ -5,5 +5,5 @@
       <parent link="base_link"/>
       <child link="imu_link"/>
-      <origin xyz="-.138 0 .02" rpy="0 1.57 0"/>
+      <origin xyz="0.01 0 .0916" rpy="0 1.57 0"/>
     </joint>
   </xacro:macro>

Commit message: Modified ekf stuff for absolute heading and fixed yaw_offset

File: urdf/sensors/imu.urdf.xacro (robot description, xacro)
@@ -5,5 +5,5 @@
       <parent link="base_link"/>
       <child link="imu_link"/>
-      <origin xyz="0.01 0 .0916" rpy="0 1.57 0"/>
+      <origin xyz="0 0 .2032" rpy="-0.175 -0.105 0"/>
     </joint>
   </xacro:macro>

Commit message: Car works

File: urdf/sensors/imu.urdf.xacro (robot description, xacro)
@@ -5,5 +5,5 @@
       <parent link="base_link"/>
       <child link="imu_link"/>
-      <origin xyz="0 0 .2032" rpy="-0.175 -0.105 0"/>
+      <origin xyz="0 0 .2032" rpy="-0.175 -0.105 3.14"/>
     </joint>
   </xacro:macro>

Commit message: Initial commit

File: urdf/sensors/imu.urdf.xacro (robot description, xacro)
@@ -5,5 +5,5 @@
       <parent link="base_link"/>
       <child link="imu_link"/>
-      <origin xyz="0 0 .2032" rpy="-0.175 -0.105 3.14"/>
+      <origin xyz="0.08161 0.0551 .15748" rpy="0 0 1.57"/>
     </joint>
   </xacro:macro>
